File: PDH_photodiode.sch (KiCad schematic (older format))
At the start: 34 parts, among them J1 ±5V-Supply, J2 AC Out, J3 DC Out, U1 LT3032, U2 LTC6269-10

Commit message: Changed 100n Caps to group standard
Parts:
- C12, C9: MFN Wurth Electronics -> Kemet; PN 885012206071 -> C0603C104K5RECAUTO
Changed lines of the file:
@@
 $EndDescr
-$Comp
-L Device:C_Small C1
-U 1 1 599D549D
-P 4000 4750
-F 0 "C1" H 4010 4820 50  0000 L CNN
-F 1 "10u" H 4010 4670 50  0000 L CNN
-F 2 "Capacitor_SMD:C_1210_3225Metric" H 4000 4750 50  0001 C CNN
-F 3 "" H 4000 4750 50  0001 C CNN
-F 4 "Taiyo Yuden" H 4000 4750 60  0001 C CNN "MFN"
-F 5 "UMR325AC7106MM-P" H 4000 4750 50  0001 C CNN "PN"
-	1    4000 4750
-	1    0    0    -1
-$EndComp
 $Comp
 L Device:C_Small C2
@@
 F 5 "UMR325AC7106MM-P" H 4000 5450 50  0001 C CNN "PN"
 	1    4000 5450
-	1    0    0    -1
-$EndComp
-$Comp
-L Device:C_Small C3
-U 1 1 599D5BFB
-P 6150 4900
-F 0 "C3" H 6160 4970 50  0000 L CNN
-F 1 "10n" H 6160 4820 50  0000 L CNN
-F 2 "Capacitor_SMD:C_0603_1608Metric" H 6150 4900 50  0001 C CNN
-F 3 "" H 6150 4900 50  0001 C CNN
-F 4 "Murata Electronics" H 6150 4900 60  0001 C CNN "MFN"
-F 5 "GRM1885C1H103JA01D" H 6150 4900 50  0001 C CNN "PN"
-	1    6150 4900
-	1    0    0    -1
-$EndComp
-$Comp
-L Device:C_Small C4
-U 1 1 599D5C38
-P 6150 5300
-F 0 "C4" H 6160 5370 50  0000 L CNN
-F 1 "10n" H 6160 5220 50  0000 L CNN
-F 2 "Capacitor_SMD:C_0603_1608Metric" H 6150 5300 50  0001 C CNN
-F 3 "" H 6150 5300 50  0001 C CNN
-F 4 "Murata Electronics" H 6150 5300 60  0001 C CNN "MFN"
-F 5 "GRM1885C1H103JA01D" H 6150 5300 50  0001 C CNN "PN"
-	1    6150 5300
 	1    0    0    -1
 $EndComp
@@
 F 2 "Capacitor_SMD:C_0603_1608Metric" H 4050 1950 50  0001 C CNN
 F 3 "" H 4050 1950 50  0001 C CNN
-F 4 "Wurth Electronics" H 4050 1950 60  0001 C CNN "MFN"
-F 5 "885012206071" H 4050 1950 50  0001 C CNN "PN"
+F 4 "Kemet" H 4050 1950 60  0001 C CNN "MFN"
+F 5 "C0603C104K5RECAUTO" H 4050 1950 50  0001 C CNN "PN"
 	1    4050 1950
 	-1   0    0    1
@@
 F 2 "Capacitor_SMD:C_0603_1608Metric" H 4850 2900 50  0001 C CNN
 F 3 "" H 4850 2900 50  0001 C CNN
-F 4 "Wurth Electronics" H 4850 2900 60  0001 C CNN "MFN"
-F 5 "" H 4850 2900 60  0001 C CNN "MFP"
-F 6 "885012206071" H 4850 2900 50  0001 C CNN "PN"
+F 4 "Kemet" H 4850 2900 60  0001 C CNN "MFN"
+F 5 "C0603C104K5RECAUTO" H 4850 2900 50  0001 C CNN "PN"
 	1    4850 2900
 	1    0    0    1
@@
 Text Notes 6300 900  0    60   ~ 0
 Use C1 (and R11) for \noptional low pass filtering.
+$Comp
+L Device:C_Small C1
+U 1 1 599D549D
+P 4000 4750
+F 0 "C1" H 4010 4820 50  0000 L CNN
+F 1 "10u" H 4010 4670 50  0000 L CNN
+F 2 "Capacitor_SMD:C_1210_3225Metric" H 4000 4750 50  0001 C CNN
+F 3 "" H 4000 4750 50  0001 C CNN
+F 4 "Taiyo Yuden" H 4000 4750 60  0001 C CNN "MFN"
+F 5 "UMR325AC7106MM-P" H 4000 4750 50  0001 C CNN "PN"
+	1    4000 4750
+	1    0    0    -1
+$EndComp
+$Comp
+L Device:C_Small C4
+U 1 1 599D5C38
+P 6150 5300
+F 0 "C4" H 6160 5370 50  0000 L CNN
+F 1 "10n" H 6160 5220 50  0000 L CNN
+F 2 "Capacitor_SMD:C_0603_1608Metric" H 6150 5300 50  0001 C CNN
+F 3 "" H 6150 5300 50  0001 C CNN
+F 4 "Murata Electronics" H 6150 5300 60  0001 C CNN "MFN"
+F 5 "GRM1885C1H103JA01D" H 6150 5300 50  0001 C CNN "PN"
+	1    6150 5300
+	1    0    0    -1
+$EndComp
+$Comp
+L Device:C_Small C3
+U 1 1 599D5BFB
+P 6150 4900
+F 0 "C3" H 6160 4970 50  0000 L CNN
+F 1 "10n" H 6160 4820 50  0000 L CNN
+F 2 "Capacitor_SMD:C_0603_1608Metric" H 6150 4900 50  0001 C CNN
+F 3 "" H 6150 4900 50  0001 C CNN
+F 4 "Murata Electronics" H 6150 4900 60  0001 C CNN "MFN"
+F 5 "GRM1885C1H103JA01D" H 6150 4900 50  0001 C CNN "PN"
+	1    6150 4900
+	1    0    0    -1
+$EndComp
 $EndSCHEMATC

Commit message: Replaced R2 and R7 with a 100k resistor (was 105k). The supply voltage therefore drops to 2.44 V (from 2.5 V)
Parts:
- R2, R7: value 105k -> 100k; PN RR0816P-1053-D-03D -> RR0816P-104-D
- R8: MFN Vishay/Beyschlag -> Vishay; PN MCT06030Z0000ZP500 -> CRCW08050000Z0EA
Other:
- note added: "-2.44 V"
- note added: "2.44 V"
Changed lines of the file:
@@
 P 6450 4700
 F 0 "R2" H 6509 4746 50  0000 L CNN
-F 1 "105k" H 6509 4655 50  0000 L CNN
+F 1 "100k" H 6509 4655 50  0000 L CNN
 F 2 "Resistor_SMD:R_0603_1608Metric" H 6450 4700 50  0001 C CNN
 F 3 "~" H 6450 4700 50  0001 C CNN
 F 4 "Susumu" H 6450 4700 50  0001 C CNN "MFN"
-F 5 "RR0816P-1053-D-03D" H 6450 4700 50  0001 C CNN "PN"
+F 5 "RR0816P-104-D" H 6450 4700 50  0001 C CNN "PN"
 	1    6450 4700
 	1    0    0    -1
@@
 P 6450 5500
 F 0 "R7" H 6509 5546 50  0000 L CNN
-F 1 "105k" H 6509 5455 50  0000 L CNN
+F 1 "100k" H 6509 5455 50  0000 L CNN
 F 2 "Resistor_SMD:R_0603_1608Metric" H 6450 5500 50  0001 C CNN
 F 3 "~" H 6450 5500 50  0001 C CNN
 F 4 "Susumu" H 6450 5500 50  0001 C CNN "MFN"
-F 5 "RR0816P-1053-D-03D" H 6450 5500 50  0001 C CNN "PN"
+F 5 "RR0816P-104-D" H 6450 5500 50  0001 C CNN "PN"
 	1    6450 5500
 	1    0    0    -1
@@
 F 2 "Resistor_SMD:R_0603_1608Metric" H 6600 2450 50  0001 C CNN
 F 3 "" H 6600 2450 50  0001 C CNN
-F 4 "Vishay/Beyschlag" H 6600 2450 60  0001 C CNN "MFN"
-F 5 "MCT06030Z0000ZP500" H 6600 2450 50  0001 C CNN "PN"
+F 4 "Vishay" H 6600 2450 60  0001 C CNN "MFN"
+F 5 "CRCW08050000Z0EA" H 6600 2450 50  0001 C CNN "PN"
 	1    6600 2450
 	0    -1   -1   0
 $EndComp
-Wire Wire Line
-	6700 2450 6850 2450
 Connection ~ 6850 2450
-Wire Wire Line
-	6500 2450 6300 2450
 Connection ~ 6300 2450
 $Comp
@@
 	1    0    0    -1
 $EndComp
+Text Notes 6850 4550 0    60   ~ 0
+2.44 V
+Text Notes 6800 5750 0    60   ~ 0
+-2.44 V
+Wire Wire Line
+	6700 2450 6850 2450
+Wire Wire Line
+	6300 2450 6500 2450
 $EndSCHEMATC

Commit message: Replace R8=0 by NC jumper
Parts:
- added JP1: Jumper_NC, Jumper:SolderJumper-2_P1.3mm_Bridged_RoundedPad1.0x1.5mm, symbol Device:Jumper_NC_Small
- R8: value 0 -> DNF; Config (none) -> DNF; MFN Vishay -> (none); PN CRCW08050000Z0EA -> (none)
Connections:
- wire segments 110 -> 114
Other:
- moved on the sheet: R8
Changed lines of the file:
@@
 L Device:R_Small R8
 U 1 1 6039FA2B
-P 6600 2450
-F 0 "R8" H 6630 2470 50  0000 L CNN
-F 1 "0" H 6630 2410 50  0000 L CNN
-F 2 "Resistor_SMD:R_0603_1608Metric" H 6600 2450 50  0001 C CNN
-F 3 "" H 6600 2450 50  0001 C CNN
-F 4 "Vishay" H 6600 2450 60  0001 C CNN "MFN"
-F 5 "CRCW08050000Z0EA" H 6600 2450 50  0001 C CNN "PN"
-	1    6600 2450
+P 6600 2150
+F 0 "R8" H 6630 2170 50  0000 L CNN
+F 1 "DNF" H 6630 2110 50  0000 L CNN
+F 2 "Resistor_SMD:R_0603_1608Metric" H 6600 2150 50  0001 C CNN
+F 3 "" H 6600 2150 50  0001 C CNN
+F 4 "" H 6600 2150 60  0001 C CNN "MFN"
+F 5 "" H 6600 2150 50  0001 C CNN "PN"
+F 6 "DNF" H 6600 2150 50  0001 C CNN "Config"
+	1    6600 2150
 	0    -1   -1   0
 $EndComp
@@
 Wire Wire Line
 	6300 2450 6500 2450
+$Comp
+L Device:Jumper_NC_Small JP1
+U 1 1 613009E4
+P 6600 2450
+F 0 "JP1" H 6600 2662 50  0000 C CNN
+F 1 "Jumper_NC" H 6600 2571 50  0000 C CNN
+F 2 "Jumper:SolderJumper-2_P1.3mm_Bridged_RoundedPad1.0x1.5mm" H 6600 2450 50  0001 C CNN
+F 3 "~" H 6600 2450 50  0001 C CNN
+F 4 "DNF" H 6600 2450 50  0001 C CNN "Config"
+	1    6600 2450
+	1    0    0    -1
+$EndComp
+Wire Wire Line
+	6700 2150 6850 2150
+Wire Wire Line
+	6850 2150 6850 2450
+Wire Wire Line
+	6500 2150 6300 2150
+Wire Wire Line
+	6300 2150 6300 2450
 $EndSCHEMATC
