File: PDH_photodiode.sch (KiCad schematic (older format))
At the start: 35 parts, among them J1 ±5V-Supply, J2 AC Out, J3 DC Out, U1 LT3032, U2 LTC6269-10

Commit message: Add buffer for DC output
Note: The buffer amplifier (LTC6228) limits the output slew rate.
Parts:
- added C13, C14: 100n, Capacitor_SMD:C_0603_1608Metric, symbol Device:C_Small
- added U3: LTC6228HS8, Package_SO:SO-8_3.9x4.9mm_P1.27mm, symbol Amplifier_Operational:LTC6228xS8
Connections:
- wire segments 114 -> 130
Other:
- moved on the sheet: C11, J3, R11
Changed lines of the file:
@@
 Sheet 1 1
 Title "PDH photodiode"
-Date "2021-02-19"
-Rev "1.1"
+Date "2021-09-01"
+Rev "1.2"
 Comp "Atoms-Photons-Quanta, Institut für Angewandte Physik, TU Darmstadt"
 Comment1 "Tilman Preuschoff"
@@
 L power:GND #PWR0105
 U 1 1 60382792
-P 7450 1550
-F 0 "#PWR0105" H 7450 1300 50  0001 C CNN
-F 1 "GND" H 7450 1400 50  0000 C CNN
-F 2 "" H 7450 1550 50  0001 C CNN
-F 3 "" H 7450 1550 50  0001 C CNN
-	1    7450 1550
+P 9800 1550
+F 0 "#PWR0105" H 9800 1300 50  0001 C CNN
+F 1 "GND" H 9800 1400 50  0000 C CNN
+F 2 "" H 9800 1550 50  0001 C CNN
+F 3 "" H 9800 1550 50  0001 C CNN
+	1    9800 1550
 	1    0    0    -1
 $EndComp
@@
 L Device:R_Small R11
 U 1 1 6038279E
-P 5950 1200
-F 0 "R11" H 5980 1220 50  0000 L CNN
-F 1 "49.9" H 5980 1160 50  0000 L CNN
-F 2 "Resistor_SMD:R_1206_3216Metric" H 5950 1200 50  0001 C CNN
-F 3 "" H 5950 1200 50  0001 C CNN
-F 4 "Yageo" H 5950 1200 60  0001 C CNN "MFN"
-F 5 "RT1206FRE0749R9L" H 5950 1200 50  0001 C CNN "PN"
-	1    5950 1200
+P 8300 1200
+F 0 "R11" H 8330 1220 50  0000 L CNN
+F 1 "49.9" H 8330 1160 50  0000 L CNN
+F 2 "Resistor_SMD:R_1206_3216Metric" H 8300 1200 50  0001 C CNN
+F 3 "" H 8300 1200 50  0001 C CNN
+F 4 "Yageo" H 8300 1200 60  0001 C CNN "MFN"
+F 5 "RT1206FRE0749R9L" H 8300 1200 50  0001 C CNN "PN"
+	1    8300 1200
 	0    1    1    0
 $EndComp
@@
 L Device:C_Small C11
 U 1 1 603827A9
-P 6300 1400
-F 0 "C11" H 6310 1470 50  0000 L CNN
-F 1 "DNF" H 6310 1320 50  0000 L CNN
-F 2 "Capacitor_SMD:C_0603_1608Metric" H 6300 1400 50  0001 C CNN
-F 3 "" H 6300 1400 50  0001 C CNN
-F 4 "DNF" H 6300 1400 50  0001 C CNN "Config"
-	1    6300 1400
-	1    0    0    -1
-$EndComp
-Wire Wire Line
-	6300 1500 6300 1550
-Wire Wire Line
-	5450 1200 5850 1200
-Wire Wire Line
-	6050 1200 6300 1200
-Wire Wire Line
-	6300 1300 6300 1200
-Connection ~ 6300 1200
-Wire Wire Line
-	7450 1400 7450 1550
-Wire Wire Line
-	6300 1200 7250 1200
+P 8650 1400
+F 0 "C11" H 8660 1470 50  0000 L CNN
+F 1 "DNF" H 8660 1320 50  0000 L CNN
+F 2 "Capacitor_SMD:C_0603_1608Metric" H 8650 1400 50  0001 C CNN
+F 3 "" H 8650 1400 50  0001 C CNN
+F 4 "DNF" H 8650 1400 50  0001 C CNN "Config"
+	1    8650 1400
+	1    0    0    -1
+$EndComp
+Wire Wire Line
+	8650 1500 8650 1550
+Wire Wire Line
+	7800 1200 8200 1200
+Wire Wire Line
+	8400 1200 8650 1200
+Wire Wire Line
+	8650 1300 8650 1200
+Connection ~ 8650 1200
+Wire Wire Line
+	9800 1400 9800 1550
+Wire Wire Line
+	8650 1200 9600 1200
 $Comp
 L power:GND #PWR0106
 U 1 1 603827BA
-P 6300 1550
-F 0 "#PWR0106" H 6300 1300 50  0001 C CNN
-F 1 "GND" H 6300 1400 50  0000 C CNN
-F 2 "" H 6300 1550 50  0001 C CNN
-F 3 "" H 6300 1550 50  0001 C CNN
-	1    6300 1550
-	1    0    0    -1
-$EndComp
-Wire Wire Line
-	5450 1200 5450 2450
+P 8650 1550
+F 0 "#PWR0106" H 8650 1300 50  0001 C CNN
+F 1 "GND" H 8650 1400 50  0000 C CNN
+F 2 "" H 8650 1550 50  0001 C CNN
+F 3 "" H 8650 1550 50  0001 C CNN
+	1    8650 1550
+	1    0    0    -1
+$EndComp
 Connection ~ 5450 2450
 Wire Wire Line
@@
 L Connector:Conn_Coaxial J3
 U 1 1 603824EE
-P 7450 1200
-F 0 "J3" H 7450 1350 50  0000 C CNN
-F 1 "DC Out" V 7550 1200 50  0000 C CNN
-F 2 "Connector_Coaxial:SMA_Amphenol_901-144_Vertical" H 7450 1200 50  0001 C CNN
-F 3 "" H 7450 1200 50  0001 C CNN
-F 4 "Amphenol" H 7450 1200 50  0001 C CNN "MFN"
-F 5 "901-144" H 7450 1200 50  0001 C CNN "PN"
-	1    7450 1200
+P 9800 1200
+F 0 "J3" H 9800 1350 50  0000 C CNN
+F 1 "DC Out" V 9900 1200 50  0000 C CNN
+F 2 "Connector_Coaxial:SMA_Amphenol_901-144_Vertical" H 9800 1200 50  0001 C CNN
+F 3 "" H 9800 1200 50  0001 C CNN
+F 4 "Amphenol" H 9800 1200 50  0001 C CNN "MFN"
+F 5 "901-144" H 9800 1200 50  0001 C CNN "PN"
+	1    9800 1200
 	1    0    0    -1
 $EndComp
@@
 NoConn ~ 4600 2250
 NoConn ~ 7850 2750
-Text Notes 6300 900  0    60   ~ 0
+Text Notes 8650 900  0    60   ~ 0
 Use C1 (and R11) for \noptional low pass filtering.
 $Comp
@@
 Wire Wire Line
 	6300 2150 6300 2450
+$Comp
+L Amplifier_Operational:LTC6228xS8 U3
+U 1 1 6132A7C7
+P 7500 1200
+F 0 "U3" H 7500 1681 50  0000 C CNN
+F 1 "LTC6228HS8" H 7700 1550 50  0000 C CNN
+F 2 "Package_SO:SO-8_3.9x4.9mm_P1.27mm" H 7500 600 50  0001 C CNN
+F 3 "https://www.analog.com/media/en/technical-documentation/data-sheets/LTC6228-6229.pdf" H 7500 1200 50  0001 C CNN
+F 4 "Analog Devices" H 7500 1200 50  0001 C CNN "MFN"
+F 5 "LTC6228HS8#PBF" H 7500 1200 50  0001 C CNN "PN"
+	1    7500 1200
+	1    0    0    -1
+$EndComp
+Text GLabel 7400 700  1    60   Input ~ 0
+V+
+Wire Wire Line
+	7400 1500 7400 1550
+Connection ~ 7400 1550
+$Comp
+L Device:C_Small C14
+U 1 1 6133209C
+P 7050 1650
+F 0 "C14" H 7060 1720 50  0000 L CNN
+F 1 "100n" H 7060 1570 50  0000 L CNN
+F 2 "Capacitor_SMD:C_0603_1608Metric" H 7050 1650 50  0001 C CNN
+F 3 "" H 7050 1650 50  0001 C CNN
+F 4 "Kemet" H 7050 1650 60  0001 C CNN "MFN"
+F 5 "C0603C104K5RECAUTO" H 7050 1650 50  0001 C CNN "PN"
+	1    7050 1650
+	-1   0    0    1
+$EndComp
+$Comp
+L power:GND #PWR0108
+U 1 1 613320A2
+P 7050 1800
+F 0 "#PWR0108" H 7050 1550 50  0001 C CNN
+F 1 "GND" H 7050 1650 50  0000 C CNN
+F 2 "" H 7050 1800 50  0001 C CNN
+F 3 "" H 7050 1800 50  0001 C CNN
+	1    7050 1800
+	-1   0    0    -1
+$EndComp
+Wire Wire Line
+	7050 1750 7050 1800
+Wire Wire Line
+	7400 1550 7400 1600
+Wire Wire Line
+	7400 1550 7050 1550
+Text GLabel 7400 1600 3    60   Input ~ 0
+V-
+$Comp
+L Device:C_Small C13
+U 1 1 6133DDFE
+P 6900 700
+F 0 "C13" H 6910 770 50  0000 L CNN
+F 1 "100n" H 6910 620 50  0000 L CNN
+F 2 "Capacitor_SMD:C_0603_1608Metric" H 6900 700 50  0001 C CNN
+F 3 "" H 6900 700 50  0001 C CNN
+F 4 "Kemet" H 6900 700 60  0001 C CNN "MFN"
+F 5 "C0603C104K5RECAUTO" H 6900 700 50  0001 C CNN "PN"
+	1    6900 700
+	-1   0    0    1
+$EndComp
+$Comp
+L power:GND #PWR0109
+U 1 1 6133E0E2
+P 6900 850
+F 0 "#PWR0109" H 6900 600 50  0001 C CNN
+F 1 "GND" H 6900 700 50  0000 C CNN
+F 2 "" H 6900 850 50  0001 C CNN
+F 3 "" H 6900 850 50  0001 C CNN
+	1    6900 850
+	1    0    0    -1
+$EndComp
+Wire Wire Line
+	6900 800  6900 850
+Wire Wire Line
+	6900 600  7150 600
+Wire Wire Line
+	7150 600  7150 800
+Wire Wire Line
+	7400 700  7400 800
+Wire Wire Line
+	7150 800  7400 800
+Connection ~ 7400 800
+Wire Wire Line
+	7400 800  7400 900
+Text GLabel 7500 1600 3    60   Input ~ 0
+V+
+Wire Wire Line
+	7500 1500 7500 1600
+Wire Wire Line
+	7800 2050 6800 2050
+Wire Wire Line
+	6800 2050 6800 1300
+Wire Wire Line
+	6800 1300 7200 1300
+Wire Wire Line
+	7800 1100 7800 2050
+Wire Wire Line
+	5450 1100 7200 1100
+Wire Wire Line
+	5450 1100 5450 2450
 $EndSCHEMATC

Commit message: Update BOM
Parts:
- J3: PN 901-144 -> 901-144-8RFX
Changed lines of the file:
@@
 F 3 "" H 9800 1200 50  0001 C CNN
 F 4 "Amphenol" H 9800 1200 50  0001 C CNN "MFN"
-F 5 "901-144" H 9800 1200 50  0001 C CNN "PN"
+F 5 "901-144-8RFX" H 9800 1200 50  0001 C CNN "PN"
 	1    9800 1200
 	1    0    0    -1
