File: KiCad/PDH_photodiode.kicad_sch (KiCad schematic)
At the start: 38 parts, among them J1 ±5V-Supply, J2 AC Out, J3 DC Out, U1 LT3032, U2 LTC6269-10, U3 LTC6228HS8

Commit message: Update to KiCad7
Parts:
- D1: footprint footprints:TO-18-3_mod -> Package_TO_SOT_THT:TO-18-3
